File: eagle/Pendent.brd (EAGLE design)
At the start: 47.5 x 40.6 mm, 39 parts, among them Q1 CMA-4544PF-W, Q2 MPSA42, Q3 8/16/20MHz, U1 MAX9814TDFN14, U2 LF50ABDT-TR, U3 ATMEGA328

Commit message: Add Push On Button
Parts:
- added D1: (no value), adafruit:SMADIODE
- added D2: Green, adafruit:CHIPLED_0805
- added Q4: (no value), adafruit:SOT23
- added R10: 1K, adafruit:R0805
- added S2: Tempo, SparkFun-Electromechanical:TACTILE-SWITCH-SMD
- C14: device SparkFun:0603-CAP -> adafruit:C0805K
- R9: value 330 -> 300
Connections:
- removed net VBATT: C8.1, U$3.P$1, U$3.P$2, U2.1
- new net N$20: D1.A, D2.A, S2.3, S2.4
- new net VBAT: Q4.3, S2.1, S2.2, U$3.P$1, U$3.P$2
- new net VIN: C8.1, D1.C, Q4.2, U2.1
- net D6: now also Q4.1
- net D7: now also D2.C, R10.2
- net GND: now also R10.1
Routing:
- net VBATT: track 57.5 -> 0.00 mm, vias 1 -> 0
- net VIN: track 0.00 -> 52.2 mm, vias 0 -> 1

Commit message: Remove non-working mosfet, switch to using power down
Parts:
- removed D1: (no value), adafruit:SMADIODE
- removed D2: Green, adafruit:CHIPLED_0805
- removed Q4: (no value), adafruit:SOT23
- removed R10: 1K, adafruit:R0805
- S2: value Tempo -> Sleep
Connections:
- removed net N$20: D1.A, D2.A, S2.3, S2.4
- removed net VBAT: Q4.3, S2.1, S2.2, U$3.P$1, U$3.P$2
- net D3: now also S2.1, S2.2; no longer R5.1
- net D6: no longer Q4.1
- net D7: no longer D2.C, R10.2
- net D9: now also R5.1
- net GND: now also S2.3, S2.4; no longer R10.1
- net VIN: now also U$3.P$1, U$3.P$2; no longer D1.C, Q4.2
Routing:
- net D3: track 4.41 -> 2.42 mm
Changed lines of the file:
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@@
 </element>
 <element name="IR" library="bg_eagle_lib" package="TOSP62XX_A" value="IR_TOSP6238TTCT-ND" x="43.5864" y="20.32" rot="R90"/>
-<element name="Q4" library="adafruit" package="SOT23" value="" x="1.27" y="-5.08"/>
-<element name="S2" library="SparkFun-Electromechanical" package="TACTILE-SWITCH-SMD" value="Tempo" x="2.54" y="-10.16">
+<element name="S2" library="SparkFun-Electromechanical" package="TACTILE-SWITCH-SMD" value="Sleep" x="2.54" y="-10.16">
 <attribute name="PROD_ID" value="SWCH-08247" x="2.54" y="-10.16" size="1.778" layer="27" display="off"/>
 </element>
-<element name="D1" library="adafruit" package="SMADIODE" value="" x="3.81" y="-16.51"/>
-<element name="D2" library="adafruit" package="CHIPLED_0805" value="Green" x="-5.08" y="-21.59"/>
-<element name="R10" library="adafruit" package="R0805" value="1K" x="-5.08" y="-27.94"/>
 </elements>
 <signals>
@@
 <via x="21.59" y="17.653" extent="1-16" drill="0.381"/>
 <via x="25.273" y="16.002" extent="1-16" drill="0.381"/>
-<contactref element="R10" pad="1"/>
+<contactref element="D3" pad="C"/>
 <contactref element="U$3" pad="GND"/>
-<contactref element="D3" pad="C"/>
+<contactref element="S2" pad="3"/>
+<contactref element="S2" pad="4"/>
 <wire x1="29.956" y1="34.544" x2="35.1536" y2="37.5412" width="0" layer="19" extent="1-1"/>
 <wire x1="33.057" y1="28.88" x2="29.956" y2="34.544" width="0" layer="19" extent="1-1"/>
@@
 <wire x1="20.32" y1="33.02" x2="24.464290625" y2="25.531090625" width="0" layer="19" extent="1-16"/>
 <wire x1="19.304" y1="34.608" x2="20.32" y2="33.02" width="0" layer="19" extent="1-16"/>
-<wire x1="-6.08" y1="-27.94" x2="3.81" y2="3.683" width="0" layer="19" extent="1-16"/>
+<wire x1="5.334" y1="-12.065" x2="3.81" y2="3.683" width="0" layer="19" extent="1-16"/>
+<wire x1="-0.254" y1="-12.065" x2="5.334" y2="-12.065" width="0" layer="19" extent="1-1"/>
 </signal>
 <signal name="VIN">
@@
 <wire x1="13.8844" y1="25.9334" x2="8.3058" y2="25.9334" width="0.6096" layer="1"/>
 <wire x1="8.3058" y1="30.48" x2="6.35" y2="30.48" width="0.508" layer="16"/>
-<contactref element="Q4" pad="2"/>
-<contactref element="D1" pad="C"/>
-<wire x1="2.22" y1="-6.18" x2="8.3058" y2="25.9334" width="0" layer="19" extent="1-16"/>
-<wire x1="1.4605" y1="-16.51" x2="2.22" y2="-6.18" width="0" layer="19" extent="1-1"/>
+<contactref element="U$3" pad="P$1"/>
+<contactref element="U$3" pad="P$2"/>
+<wire x1="32.8676" y1="30.5276" x2="34.544" y2="32.893" width="0" layer="19" extent="16-16"/>
+<wire x1="6.096" y1="32.893" x2="6.35" y2="30.48" width="0" layer="19" extent="16-16"/>
 </signal>
 <signal name="INPUT">
@@
 <wire x1="32.385" y1="23.495" x2="32.54668125" y2="23.68896875" width="0.508" layer="1"/>
 <wire x1="36.195" y1="29.845" x2="36.7284" y2="30.0134" width="0.508" layer="1"/>
+<contactref element="R5" pad="1"/>
+<wire x1="34.6456" y1="13.9794" x2="32.385" y2="23.495" width="0" layer="19" extent="1-16"/>
 </signal>
 <signal name="D8">
@@
 <signal name="D3">
 <contactref element="U3" pad="1"/>
-<contactref element="R5" pad="1"/>
 <via x="32.6136" y="13.9192" extent="1-16" drill="0.381"/>
 <wire x1="30.849625" y1="15.355571875" x2="30.872428125" y2="15.355571875" width="0.4064" layer="1"/>
@@
 <wire x1="31.6484" y1="14.5796" x2="31.9532" y2="14.5796" width="0.4064" layer="1"/>
 <wire x1="31.9532" y1="14.5796" x2="32.6136" y2="13.9192" width="0.4064" layer="1"/>
-<wire x1="34.6456" y1="13.9794" x2="32.6534" y2="13.8794" width="0.4064" layer="16"/>
 <wire x1="32.6534" y1="13.8794" x2="32.6136" y2="13.9192" width="0.4064" layer="16"/>
+<contactref element="S2" pad="1"/>
+<contactref element="S2" pad="2"/>
+<wire x1="5.334" y1="-8.255" x2="30.849625" y2="15.355571875" width="0" layer="19" extent="1-1"/>
+<wire x1="-0.254" y1="-8.255" x2="5.334" y2="-8.255" width="0" layer="19" extent="1-1"/>
 </signal>
 <signal name="D4">
@@
 <signal name="D6">
 <contactref element="U3" pad="10"/>
-<contactref element="Q4" pad="1"/>
-<wire x1="0.32" y1="-6.18" x2="34.2437375" y2="21.9919125" width="0" layer="19" extent="1-1"/>
 </signal>
 <signal name="D7">
 <contactref element="U3" pad="11"/>
-<contactref element="D2" pad="C"/>
-<contactref element="R10" pad="2"/>
-<wire x1="-5.08" y1="-20.54" x2="33.678053125" y2="22.557596875" width="0" layer="19" extent="1-1"/>
-<wire x1="-4.08" y1="-27.94" x2="-5.08" y2="-20.54" width="0" layer="19" extent="1-1"/>
 </signal>
 <signal name="D10">
@@
 <wire x1="4.1275" y1="26.035" x2="3.937" y2="25.8826" width="0.254" layer="1"/>
 </signal>
-<signal name="VBAT">
-<contactref element="Q4" pad="3"/>
-<contactref element="S2" pad="1"/>
-<contactref element="S2" pad="2"/>
-<contactref element="U$3" pad="P$2"/>
-<contactref element="U$3" pad="P$1"/>
-<wire x1="6.096" y1="32.893" x2="34.544" y2="32.893" width="0" layer="19" extent="16-16"/>
-<wire x1="1.27" y1="-3.98" x2="6.096" y2="32.893" width="0" layer="19" extent="1-16"/>
-<wire x1="-0.254" y1="-8.255" x2="1.27" y2="-3.98" width="0" layer="19" extent="1-1"/>
-<wire x1="5.334" y1="-8.255" x2="-0.254" y2="-8.255" width="0" layer="19" extent="1-1"/>
-</signal>
-<signal name="N$20">
-<contactref element="S2" pad="4"/>
-<contactref element="S2" pad="3"/>
-<contactref element="D1" pad="A"/>
-<contactref element="D2" pad="A"/>
-<wire x1="-0.254" y1="-12.065" x2="-5.08" y2="-22.64" width="0" layer="19" extent="1-1"/>
-<wire x1="5.334" y1="-12.065" x2="-0.254" y2="-12.065" width="0" layer="19" extent="1-1"/>
-<wire x1="6.1595" y1="-16.51" x2="5.334" y2="-12.065" width="0" layer="19" extent="1-1"/>
-</signal>
 </signals>
